File: PCB Design/Digi2_Act8085.kicad_sch (KiCad schematic)
At the start: 22 parts, among them U1 8085A, U11 IR4301, U12 74HC238, U2 Barrel_Jack, U3 L7805, Y1 3MHz

Commit message: Remove IC not included
Parts:
- removed U11: IR4301, Package_DFN_QFN:Infineon_PQFN-22-15-4EP_6x5mm_P0.65mm, symbol Amplifier_Audio:IR4301
- removed U12: 74HC238, symbol 74xx_IEEE:74HC238
Changed lines of the file:
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@@
-	(wire
-		(pts
-			(xy 116.84 66.04) (xy 116.84 133.35)
-		)
-		(stroke
-			(width 0)
-			(type default)
-		)
-	)
 	(wire
 		(pts
@@
 	(wire
 		(pts
-			(xy 123.19 105.41) (xy 123.19 50.8)
-		)
-		(stroke
-			(width 0)
-			(type default)
-		)
-	)
-	(wire
-		(pts
 			(xy 86.36 88.9) (xy 100.33 88.9)
 		)
@@
 	(wire
 		(pts
-			(xy 134.62 66.04) (xy 116.84 66.04)
-		)
-		(stroke
-			(width 0)
-			(type default)
-		)
-	)
-	(wire
-		(pts
 			(xy 86.36 111.76) (xy 100.33 111.76)
 		)
@@
 	(wire
 		(pts
-			(xy 116.84 133.35) (xy 123.19 133.35)
-		)
-		(stroke
-			(width 0)
-			(type default)
-		)
-	)
-	(wire
-		(pts
 			(xy 237.49 52.07) (xy 237.49 57.15)
 		)
@@
 		(pts
 			(xy 251.46 39.37) (xy 251.46 44.45)
-		)
-		(stroke
-			(width 0)
-			(type default)
-		)
-	)
-	(wire
-		(pts
-			(xy 123.19 50.8) (xy 134.62 50.8)
 		)
 		(stroke
@@
 	)
 	(symbol
-		(lib_id "74xx_IEEE:74HC238")
-		(at 143.51 115.57 0)
-		(unit 1)
-		(exclude_from_sim no)
-		(in_bom yes)
-		(on_board yes)
-		(dnp no)
-		(fields_autoplaced yes)
-		(property "Reference" "U12"
-			(at 145.7041 95.25 0)
-			(effects
-				(font
-					(size 1.27 1.27)
-				)
-				(justify left)
-			)
-		)
-		(property "Value" "74HC238"
-			(at 145.7041 97.79 0)
-			(effects
-				(font
-					(size 1.27 1.27)
-				)
-				(justify left)
-			)
-		)
-		(property "Footprint" ""
-			(at 143.51 115.57 0)
-			(effects
-				(font
-					(size 1.27 1.27)
-				)
-				(hide yes)
-			)
-		)
-		(property "Datasheet" ""
-			(at 143.51 115.57 0)
-			(effects
-				(font
-					(size 1.27 1.27)
-				)
-				(hide yes)
-			)
-		)
-		(property "Description" ""
-			(at 143.51 115.57 0)
-			(effects
-				(font
-					(size 1.27 1.27)
-				)
-				(hide yes)
-			)
-		)
-		(pin "10"
-		)
-		(pin "8"
-		)
-		(pin "6"
-		)
-		(pin "4"
-		)
-		(pin "11"
-		)
-		(pin "13"
-		)
-		(pin "9"
-		)
-		(pin "16"
-		)
-		(pin "2"
-		)
-		(pin "5"
-		)
-		(pin "15"
-		)
-		(pin "14"
-		)
-		(pin "7"
-		)
-		(pin "12"
-		)
-		(pin "3"
-		)
-		(pin "1"
-		)
-		(instances
-			(project "Digi2_Act8085"
-				(path "/da5f4034-ebed-4d21-8fe0-a4910c0c98b0"
-					(reference "U12")
-					(unit 1)
-				)
-			)
-		)
-	)
-	(symbol
 		(lib_id "power:PWR_FLAG")
 		(at 179.07 57.15 90)
@@
 					(unit 1)
 				)
-			)
-		)
-	)
-	(symbol
-		(lib_id "Amplifier_Audio:IR4301")
-		(at 144.78 66.04 0)
-		(unit 1)
-		(exclude_from_sim no)
-		(in_bom yes)
-		(on_board yes)
-		(dnp no)
-		(fields_autoplaced yes)
-		(property "Reference" "U11"
-			(at 152.0541 43.18 0)
-			(effects
-				(font
-					(size 1.27 1.27)
-				)
-				(justify left)
-			)
-		)
-		(property "Value" "IR4301"
-			(at 152.0541 45.72 0)
-			(effects
-				(font
-					(size 1.27 1.27)
-				)
-				(justify left)
-			)
-		)
-		(property "Footprint" "Package_DFN_QFN:Infineon_PQFN-22-15-4EP_6x5mm_P0.65mm"
-			(at 144.78 66.04 0)
-			(effects
-				(font
-					(size 1.27 1.27)
-					(italic yes)
-				)
-				(hide yes)
-			)
-		)
-		(property "Datasheet" "https://www.infineon.com/dgdl/ir4301.pdf?fileId=5546d462533600a4015355d5fc691819"
-			(at 144.78 66.04 0)
-			(effects
-				(font
-					(size 1.27 1.27)
-				)
-				(hide yes)
-			)
-		)
-		(property "Description" "PowIRaudio Integrated Analog Input Class D Audio Amplifier, 160W/4ohm, 80V, PQFN-22"
-			(at 144.78 66.04 0)
-			(effects
-				(font
-					(size 1.27 1.27)
-				)
-				(hide yes)
-			)
-		)
-		(pin "11"
-		)
-		(pin "14"
-		)
-		(pin "3"
-		)
-		(pin "9"
-		)
-		(pin "13"
-		)
-		(pin "5"
-		)
-		(pin "15"
-		)
-		(pin "1"
-		)
-		(pin "12"
-		)
-		(pin "4"
-		)
-		(pin "7"
-		)
-		(pin "8"
-		)
-		(pin "2"
-		)
-		(pin "10"
-		)
-		(pin "6"
-		)
-		(instances
-			(project "Digi2_Act8085"
-				(path "/da5f4034-ebed-4d21-8fe0-a4910c0c98b0"
-					(reference "U11")
-					(unit 1)
-				)

Commit message: Add ground
Parts:
- added U11: IR4301, Package_DFN_QFN:Infineon_PQFN-22-15-4EP_6x5mm_P0.65mm, symbol Amplifier_Audio:IR4301
- added U12: LM4810, Package_SO:TSSOP-8_3x3mm_P0.65mm, symbol Amplifier_Audio:LM4810
Connections:
- net GND: now also U12.4 (GND), U12.5 (SHDN)
- new net: U11.7 (VSS), U12.2 (VIN1)
- new net: U11.15 (COM), U11.9 (COM)

Commit message: Remove Not needed
Parts:
- removed U11: IR4301, Package_DFN_QFN:Infineon_PQFN-22-15-4EP_6x5mm_P0.65mm, symbol Amplifier_Audio:IR4301
- removed U12: LM4810, Package_SO:TSSOP-8_3x3mm_P0.65mm, symbol Amplifier_Audio:LM4810

Commit message: Updated PCB and Footprint
Parts:
- C1, C11: footprint Capacitor_THT:CP_Radial_D8.0mm_P3.50mm -> Capacitor_THT:CP_Radial_D5.0mm_P2.50mm
- C10: footprint Capacitor_THT:CP_Radial_D8.0mm_P3.50mm -> Capacitor_THT:CP_Radial_D4.0mm_P2.00mm
- C12: footprint Capacitor_THT:CP_Radial_D8.0mm_P3.50mm -> Capacitor_THT:C_Disc_D4.3mm_W1.9mm_P5.00mm
Changed lines of the file:
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@@
 			)
 		)
-		(property "Footprint" "Capacitor_THT:CP_Radial_D8.0mm_P3.50mm"
+		(property "Footprint" "Capacitor_THT:C_Disc_D4.3mm_W1.9mm_P5.00mm"
 			(at 43.18 127 0)
 			(effects
@@
 			)
 		)
-		(property "Footprint" "Capacitor_THT:CP_Radial_D8.0mm_P3.50mm"
+		(property "Footprint" "Capacitor_THT:CP_Radial_D5.0mm_P2.50mm"
 			(at 36.83 44.45 0)
 			(effects
@@
 			)
 		)
-		(property "Footprint" "Capacitor_THT:CP_Radial_D8.0mm_P3.50mm"
+		(property "Footprint" "Capacitor_THT:CP_Radial_D5.0mm_P2.50mm"
 			(at 252.4252 54.61 0)
 			(effects
@@
 			)
 		)
-		(property "Footprint" "Capacitor_THT:CP_Radial_D8.0mm_P3.50mm"
+		(property "Footprint" "Capacitor_THT:CP_Radial_D4.0mm_P2.00mm"
 			(at 223.2152 54.61 0)
 			(effects
