File: PCB Design/Digi2_Act8085.kicad_pcb (KiCad board)
At the start: 2 copper layers, 27 parts, among them U1 8085A, U10 8255, U2 Barrel_Jack, U3 L7805, U4 2764, U5 CY6264, U6 74LS373, U7 74LS138, U8 8255, U9 8255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

Commit message: Updated PCB and Footprint
Parts:
- C1, C11: footprint Capacitor_THT:CP_Radial_D8.0mm_P3.50mm -> Capacitor_THT:CP_Radial_D5.0mm_P2.50mm
- C10: footprint Capacitor_THT:CP_Radial_D8.0mm_P3.50mm -> Capacitor_THT:CP_Radial_D4.0mm_P2.00mm
- C12: footprint Capacitor_THT:CP_Radial_D8.0mm_P3.50mm -> Capacitor_THT:C_Disc_D4.3mm_W1.9mm_P5.00mm
- moved FB1 33.4 mm to (223.0, 69.0)
- moved C12 3.49 mm to (189.0, 59.0)

Commit message: Test Route
Routing:
- net /Memory and Peripheral Inteface/~{WR}: track 0.00 -> 22.0 mm
- net /Memory and Peripheral Inteface/~{RD}: track 0.00 -> 19.3 mm
Changed lines of the file:
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@@
 		)
 	)
+	(segment
+		(start 130.96 39.64)
+		(end 132.06 40.74)
+		(width 0.2)
+		(layer "F.Cu")
+		(net 22)
+	)
+	(segment
+		(start 114.76 39.64)
+		(end 130.96 39.64)
+		(width 0.2)
+		(layer "F.Cu")
+		(net 22)
+	)
+	(segment
+		(start 113.66 40.74)
+		(end 114.76 39.64)
+		(width 0.2)
+		(layer "F.Cu")
+		(net 22)
+	)
+	(segment
+		(start 128.9 41.675635)
+		(end 131.604365 44.38)
+		(width 0.2)
+		(layer "F.Cu")
+		(net 55)
+	)
+	(segment
+		(start 131.604365 44.38)
+		(end 143.66 44.38)
+		(width 0.2)
+		(layer "F.Cu")
+		(net 55)
+	)
+	(segment
+		(start 143.66 44.38)
+		(end 147.3 40.74)
+		(width 0.2)
+		(layer "F.Cu")
+		(net 55)
+	)
+	(segment
+		(start 128.9 40.74)
+		(end 128.9 41.675635)
+		(width 0.2)
+		(layer "F.Cu")
+		(net 55)
+	)
 )

Commit message: test
Routing:
- net /Memory and Peripheral Inteface/AD0: track 0.00 -> 19.3 mm
Changed lines of the file:
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@@
+	)
+	(segment
+		(start 146.2 46.92)
+		(end 147.3 45.82)
+		(width 0.2)
+		(layer "F.Cu")
+		(net 28)
+	)
+	(segment
+		(start 130 46.92)
+		(end 146.2 46.92)
+		(width 0.2)
+		(layer "F.Cu")
+		(net 28)
+	)
+	(segment
+		(start 128.9 45.82)
+		(end 130 46.92)
+		(width 0.2)
+		(layer "F.Cu")
+		(net 28)
 	)
 	(segment

Commit message: test
Routing:
- net /Memory and Peripheral Inteface/AD0: track 19.3 -> 3.11 mm
Changed lines of the file:
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@@
-	)
-	(segment
-		(start 130 46.92)
-		(end 146.2 46.92)
-		(width 0.2)
-		(layer "F.Cu")
-		(net 28)
 	)
 	(segment

Commit message: test
Routing:
- net /Memory and Peripheral Inteface/AD0: track 3.11 -> 19.8 mm
Changed lines of the file:
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@@
 	)
 	(segment
-		(start 146.2 46.92)
+		(start 145.62 47.5)
 		(end 147.3 45.82)
 		(width 0.2)
 		(layer "F.Cu")
+		(net 28)
+	)
+	(segment
+		(start 144.5 47.5)
+		(end 145.62 47.5)
+		(width 0.2)
+		(layer "F.Cu")
+		(net 28)
+	)
+	(segment
+		(start 130 46.92)
+		(end 143.92 46.92)
+		(width 0.2)
+		(layer "F.Cu")
+		(net 28)
+	)
+	(segment
+		(start 143.92 46.92)
+		(end 144.5 47.5)
+		(width 0.2)
+		(layer "F.Cu")
