File: PCB Design/Digi2_Act8085.kicad_pcb (KiCad board)
At the start: 2 copper layers, 27 parts, among them U1 8085A, U10 8255, U2 Barrel_Jack, U3 L7805, U4 2764, U5 CY6264, U6 74LS373, U7 74LS138, U8 8255, U9 8255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

Commit message: test
Parts:
- moved U6 30.2 mm to (84.8, 78.3)
- moved U7 30.2 mm to (96.5, 78.3)
- moved FB1 20.5 mm to (236.5, 70.0)
- moved Y1 20.5 mm to (223.1, 32.9)
- moved C3 20.5 mm to (212.5, 34.7)
- moved C5 20.5 mm to (212.5, 41.6)
- moved C7 20.5 mm to (212.5, 48.5)
- moved C8 20.5 mm to (212.5, 52.0)
- moved D1 20.5 mm to (223.2, 51.6)
- moved D2 20.5 mm to (213.3, 60.5)
- moved U2 20.5 mm to (226.4, 71.6)
- moved U3 20.5 mm to (222.3, 40.1)
- moved C2 20.5 mm to (212.5, 31.2)
- moved C4 20.5 mm to (212.5, 38.1)
- moved C6 20.5 mm to (212.5, 45.0)
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Routing:
- net /Memory and Peripheral Inteface/A2: track 0.00 -> 28.8 mm
- net /Memory and Peripheral Inteface/A12: track 0.00 -> 19.8 mm
Changed lines of the file:
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@@
 	(footprint "Capacitor_THT:C_Disc_D4.3mm_W1.9mm_P5.00mm"
 		(layer "F.Cu")
-		(at 232.575 27.19)
+		(at 212.5 31.25)
 		(descr "C, Disc series, Radial, pin pitch=5.00mm, , diameter*width=4.3*1.9mm^2, Capacitor, http://www.vishay.com/docs/45233/krseries.pdf")
 		(tags "C Disc series Radial pin pitch 5.00mm  diameter 4.3mm width 1.9mm Capacitor")
@@
 	(footprint "Package_TO_SOT_THT:TO-220-3_Vertical"
 		(layer "F.Cu")
-		(at 242.385 36.04)
+		(at 222.31 40.1)
 		(descr "TO-220-3, Vertical, RM 2.54mm, see https://www.vishay.com/docs/66542/to-220-1.pdf")
 		(tags "TO-220-3 Vertical RM 2.54mm")
@@
 	(footprint "Crystal:Crystal_HC49-U_Vertical"
 		(layer "F.Cu")
-		(at 243.175 28.79)
+		(at 223.1 32.85)
 		(descr "Crystal THT HC-49/U http://5hertz.com/pdfs/04404_D.pdf")
 		(tags "THT crystalHC-49/U")
@@
 	(footprint "Package_DIP:DIP-16_W7.62mm_Socket"
 		(layer "F.Cu")
-		(at 125.91 85.03)
+		(at 96.5 78.3)
 		(descr "16-lead though-hole mounted DIP package, row spacing 7.62 mm (300 mils), Socket")
 		(tags "THT DIP DIL PDIP 2.54mm 7.62mm 300mil Socket")
@@
 	(footprint "Package_DIP:DIP-20_W7.62mm_Socket"
 		(layer "F.Cu")
-		(at 114.16 85.03)
+		(at 84.75 78.3)
 		(descr "20-lead though-hole mounted DIP package, row spacing 7.62 mm (300 mils), Socket")
 		(tags "THT DIP DIL PDIP 2.54mm 7.62mm 300mil Socket")
@@
 	(footprint "Ferrite_THT:LairdTech_28C0236-0JW-10"
 		(layer "F.Cu")
-		(at 256.535 65.96)
+		(at 236.46 70.02)
 		(descr "Ferrite, vertical, LairdTech 28C0236-0JW-10, https://assets.lairdtech.com/home/brandworld/files/28C0236-0JW-10.pdf, JW Miller core https://www.bourns.com/products/magnetic-products/j.w.-miller-through-hole-ferrite-beads-emi-filters")
 		(tags "Ferrite vertical LairdTech 28C0236-0JW-10")
@@
 	(footprint "Capacitor_THT:C_Disc_D4.3mm_W1.9mm_P5.00mm"
 		(layer "F.Cu")
-		(at 232.575 51.34)
+		(at 212.5 55.4)
 		(descr "C, Disc series, Radial, pin pitch=5.00mm, , diameter*width=4.3*1.9mm^2, Capacitor, http://www.vishay.com/docs/45233/krseries.pdf")
 		(tags "C Disc series Radial pin pitch 5.00mm  diameter 4.3mm width 1.9mm Capacitor")
@@
 	(footprint "Capacitor_THT:C_Disc_D4.3mm_W1.9mm_P5.00mm"
 		(layer "F.Cu")
-		(at 232.575 30.64)
+		(at 212.5 34.7)
 		(descr "C, Disc series, Radial, pin pitch=5.00mm, , diameter*width=4.3*1.9mm^2, Capacitor, http://www.vishay.com/docs/45233/krseries.pdf")
 		(tags "C Disc series Radial pin pitch 5.00mm  diameter 4.3mm width 1.9mm Capacitor")
@@
 	(footprint "Capacitor_THT:C_Disc_D4.3mm_W1.9mm_P5.00mm"
 		(layer "F.Cu")
-		(at 232.575 47.89)
+		(at 212.5 51.95)
 		(descr "C, Disc series, Radial, pin pitch=5.00mm, , diameter*width=4.3*1.9mm^2, Capacitor, http://www.vishay.com/docs/45233/krseries.pdf")
 		(tags "C Disc series Radial pin pitch 5.00mm  diameter 4.3mm width 1.9mm Capacitor")
@@
 	(footprint "Capacitor_THT:C_Disc_D4.3mm_W1.9mm_P5.00mm"
 		(layer "F.Cu")
-		(at 232.575 37.54)
+		(at 212.5 41.6)
 		(descr "C, Disc series, Radial, pin pitch=5.00mm, , diameter*width=4.3*1.9mm^2, Capacitor, http://www.vishay.com/docs/45233/krseries.pdf")
 		(tags "C Disc series Radial pin pitch 5.00mm  diameter 4.3mm width 1.9mm Capacitor")
@@
 	(footprint "LED_THT:LED_D8.0mm"
 		(layer "F.Cu")
-		(at 243.225 47.5)
+		(at 223.15 51.56)
 		(descr "LED, diameter 8.0mm, 2 pins, http://cdn-reichelt.de/documents/datenblatt/A500/LED8MMGE_LED8MMGN_LED8MMRT%23KIN.pdf")
 		(tags "LED diameter 8.0mm 2 pins")
@@
 	(footprint "Connector_BarrelJack:BarrelJack_Horizontal"
 		(layer "F.Cu")
-		(at 246.5 67.5)
+		(at 226.425 71.56)
 		(descr "DC Barrel Jack")
 		(tags "Power Jack")
@@
 	(footprint "Capacitor_THT:C_Disc_D4.3mm_W1.9mm_P5.00mm"
 		(layer "F.Cu")
-		(at 232.575 34.09)
+		(at 212.5 38.15)
 		(descr "C, Disc series, Radial, pin pitch=5.00mm, , diameter*width=4.3*1.9mm^2, Capacitor, http://www.vishay.com/docs/45233/krseries.pdf")
 		(tags "C Disc series Radial pin pitch 5.00mm  diameter 4.3mm width 1.9mm Capacitor")
@@
 	(footprint "Capacitor_THT:C_Disc_D4.3mm_W1.9mm_P5.00mm"
 		(layer "F.Cu")
-		(at 232.575 40.99)
+		(at 212.5 45.05)
 		(descr "C, Disc series, Radial, pin pitch=5.00mm, , diameter*width=4.3*1.9mm^2, Capacitor, http://www.vishay.com/docs/45233/krseries.pdf")
 		(tags "C Disc series Radial pin pitch 5.00mm  diameter 4.3mm width 1.9mm Capacitor")
@@
 	(footprint "Capacitor_THT:C_Disc_D4.3mm_W1.9mm_P5.00mm"
 		(layer "F.Cu")
-		(at 232.575 44.44)
+		(at 212.5 48.5)
 		(descr "C, Disc series, Radial, pin pitch=5.00mm, , diameter*width=4.3*1.9mm^2, Capacitor, http://www.vishay.com/docs/45233/krseries.pdf")
 		(tags "C Disc series Radial pin pitch 5.00mm  diameter 4.3mm width 1.9mm Capacitor")
@@
 	(footprint "Resistor_THT:R_Axial_DIN0207_L6.3mm_D2.5mm_P7.62mm_Horizontal"
 		(layer "F.Cu")
-		(at 240.725 40.1)
+		(at 220.65 44.16)
 		(descr "Resistor, Axial_DIN0207 series, Axial, Horizontal, pin pitch=7.62mm, 0.25W = 1/4W, length*diameter=6.3*2.5mm^2, http://cdn-reichelt.de/documents/datenblatt/B400/1_4W%23YAG.pdf")
 		(tags "Resistor Axial_DIN0207 series Axial Horizontal pin pitch 7.62mm 0.25W = 1/4W length 6.3mm diameter 2.5mm")
@@
 	(footprint "Diode_THT:D_DO-201AD_P15.24mm_Horizontal"
 		(layer "F.Cu")
-		(at 233.375 56.44)
+		(at 213.3 60.5)
 		(descr "Diode, DO-201AD series, Axial, Horizontal, pin pitch=15.24mm, , length*diameter=9.5*5.2mm^2, , http://www.diodes.com/_files/packages/DO-201AD.pdf")
 		(tags "Diode DO-201AD series Axial Horizontal pin pitch 15.24mm  length 9.5mm diameter 5.2mm")
@@
 		(net 3)
 	)
+	(segment
+		(start 171.36 102.81)
+		(end 177.55 109)
+		(width 0.2)
+		(layer "F.Cu")
+		(net 23)
+	)
+	(segment
+		(start 191.36 103.86)
+		(end 190.26 102.76)
+		(width 0.2)
+		(layer "F.Cu")
+		(net 23)
+	)
+	(segment
+		(start 190.655635 109)
+		(end 191.36 108.295635)
+		(width 0.2)
+		(layer "F.Cu")
+		(net 23)
+	)
+	(segment
+		(start 191.36 108.295635)
+		(end 191.36 103.86)
+		(width 0.2)
+		(layer "F.Cu")
+		(net 23)
+	)
+	(segment
+		(start 177.55 109)
+		(end 190.655635 109)
+		(width 0.2)
+		(layer "F.Cu")
+		(net 23)
+	)
+	(segment
+		(start 171.36 87.57)
+		(end 172.46 88.67)
+		(width 0.2)
+		(layer "F.Cu")
+		(net 32)
+	)
+	(segment
+		(start 189.11 88.67)
+		(end 190.26 87.52)
+		(width 0.2)
+		(layer "F.Cu")
+		(net 32)
+	)
+	(segment
+		(start 172.46 88.67)
+		(end 189.11 88.67)
+		(width 0.2)
+		(layer "F.Cu")
+		(net 32)
+	)
 )
