File: PCB Design/Digi2_Act8085.kicad_pcb (KiCad board)
At the start: 2 copper layers, 27 parts, among them U1 8085A, U10 8255, U2 Barrel_Jack, U3 L7805, U4 2764, U5 CY6264, U6 74LS373, U7 74LS138, U8 8255, U9 8255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

Commit message: New Main File
Parts:
- moved FB1 73.6 mm to (164.0, 57.1)
- moved U2 69.1 mm to (157.7, 79.2)
- moved D2 68.5 mm to (145.6, 70.4)
- moved C2 68.0 mm to (144.8, 37.7)
- moved C3 68.0 mm to (144.8, 41.2)
- moved C4 68.0 mm to (144.8, 44.6)
- moved C5 68.0 mm to (144.8, 48.1)
- moved C6 68.0 mm to (144.8, 51.5)
- moved C7 68.0 mm to (144.8, 55.0)
- moved C8 68.0 mm to (144.8, 58.4)
- moved C9 68.0 mm to (144.8, 61.9)
- moved D1 68.0 mm to (155.4, 58.0)
- moved R1 68.0 mm to (152.9, 50.6)
- moved U3 68.0 mm to (154.6, 46.6)
- moved Y1 68.0 mm to (155.4, 39.3)
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Routing:
- net +5V: track 49.5 -> 0.00 mm
- net /Memory and Peripheral Inteface/A2: track 28.8 -> 0.00 mm
- net /Memory and Peripheral Inteface/~{WR}: track 22.0 -> 0.00 mm
- net /Memory and Peripheral Inteface/A12: track 19.8 -> 0.00 mm
- net /Memory and Peripheral Inteface/AD0: track 19.8 -> 0.00 mm
- net /Memory and Peripheral Inteface/~{RD}: track 17.8 -> 0.00 mm

Commit message: Test A
Routing:
- net Net-(U3-IN): track 0.00 -> 13.5 mm
Changed lines of the file:
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@@
 		)
 	)
+	(segment
+		(start 169.042832 57.13)
+		(end 169.042832 49.758031)
+		(width 0.2)
+		(layer "F.Cu")
+		(net 3)
+	)
+	(segment
+		(start 169.042832 49.758031)
+		(end 164.714801 45.43)
+		(width 0.2)
+		(layer "F.Cu")
+		(net 3)
+	)
 )
